Commit message: Add mass and inertia properties to URDF

File: biped_model/biped.urdf (robot description, URDF)
Before this commit: robot biped, 7 links, 6 joints
Links:
- link BODY_LINK: mass 19.0917 -> 1.404
- link LEFT_HIP_LINK: mass 1.814 -> 0.196; geometry visual mesh filename=package://biped_model/hip.STL
- link LEFT_SHIN_LINK: geometry visual mesh filename=package://biped_model/shin.STL
- link LEFT_THIGH_LINK: mass 0.762 -> 0.306; geometry visual mesh filename=package://biped_model/thigh.STL
- link RIGHT_HIP_LINK: mass 1.814 -> 0.196; geometry visual mesh filename=package://biped_model/hip.STL
- link RIGHT_SHIN_LINK: geometry visual mesh filename=package://biped_model/shin.STL
- link RIGHT_THIGH_LINK: mass 0.762 -> 0.306; geometry visual mesh filename=package://biped_model/thigh.STL
Joints:
- joint LEFT_HIP_X: origin xyz=0 0.115 -0.07185 rpy=0 0 0 -> xyz=0.055 0.0935 0.02 rpy=0 0 0
- joint LEFT_KNEE_Y: origin xyz=0 0 -0.079068 rpy=0 0 0 -> xyz=0 0 -0.3 rpy=0 0 0
- joint LEFT_THIGH_Y: origin xyz=0.035 0.015 -0.04975 rpy=0 0 0 -> xyz=-0.06 0.0345 0.0 rpy=0 0 0
- joint RIGHT_HIP_X: origin xyz=0 -0.115 -0.07185 rpy=0 0 0 -> xyz=0.055 -0.093 0.02 rpy=0 0 0
- joint RIGHT_KNEE_Y: origin xyz=0 0 -0.38 rpy=0 0 0 -> xyz=0 0 -0.3 rpy=0 0 0
- joint RIGHT_THIGH_Y: origin xyz=0.035 -0.015 -0.04975 rpy=0 0 0 -> xyz=-0.06 -0.0345 0.0 rpy=0 0 0
